File: business_card.kicad_pcb (KiCad board)
At the start: 2 copper layers, 58.4 x 31.8 mm, 12 parts, among them SW1 slide_switch_general, U1 NE556N_gen

Commit message: modified the qr code url
Parts:
- moved G*** 0.51 mm to (166.4, 101.6)
