File: archive/business_card.kicad_pcb (KiCad board)
At the start: 2 copper layers, 58.4 x 31.8 mm, 12 parts, among them SW1 slide_switch_general, U1 NE556N_gen

Commit message: major reorg
Parts:
- moved +9V 19.3 mm to (111.3, 104.1)
- moved LS1 19.3 mm to (135.9, 86.1)
- moved R1 19.3 mm to (114.3, 93.5)
- moved SW1 19.3 mm to (109.7, 84.8)
- moved U1 19.3 mm to (115.6, 90.2)
- moved - 19.3 mm to (114.8, 104.1)
- moved C2 19.3 mm to (113.3, 100.8)
- moved PR1 19.3 mm to (118.1, 78.2)
- moved G*** 19.3 mm to (154.2, 86.6)
- moved TR1 19.3 mm to (125.5, 102.1)
- moved PR2 19.3 mm to (128.3, 78.2)
- moved C1 19.3 mm to (113.3, 97.0)
Other:
- board text added: "Tristan Mullin Computer Engineering tristan.mullin1@gmail.com"
- board text removed: "Name Major Email"
